Commit message: Update fin xacros

File: uuv_gazebo_plugins/uuv_gazebo_ros_plugins/urdf/fin_snippets.xacro (robot description, xacro)
@@ -123,4 +123,51 @@
         <xacro:insert_block name="origin"/>
         <!--<axis xyz="0 0 1"/>-->
+        <axis xyz="0 -1 0"/>
+        <parent link="${parent_link}" />
+        <child link="${namespace}/fin${fin_id}" />
+    </joint>
+    <link name="${namespace}/fin${fin_id}">
+      <xacro:no_inertial />
+      <visual>
+        <origin xyz="0 0 0" rpy="0 0 0" />
+        <geometry>
+          <mesh filename="${mesh_filename}" scale="1 1 1"/>
+        </geometry>
+      </visual>
+    </link>
+    <gazebo>
+      <plugin name="${namespace}_fin${fin_id}_model" filename="libuuv_fin_ros_plugin.so">
+        <dynamics>
+          <type>FirstOrder</type>
+          <timeConstant>${fin_dynamics_time_constant}</timeConstant>
+        </dynamics>
+        <liftdrag>
+          <type>Quadratic</type>
+          <lift_constant>${lift_constant}</lift_constant>
+          <drag_constant>${drag_constant}</drag_constant>
+        </liftdrag>
+        <current_velocity_topic>${current_velocity_topic}</current_velocity_topic>
+        <fin_id>${fin_id}</fin_id>
+        <link_name>${namespace}/fin${fin_id}</link_name>
+        <joint_name>${namespace}/fin${fin_id}_joint</joint_name>
+      </plugin>
+    </gazebo>
+  </xacro:macro>
+  <xacro:macro name="hor_right_fin_quadratic_macro"
+    params="namespace
+            parent_link
+            fin_id
+            *origin
+            min_joint_limit
+            max_joint_limit
+            mesh_filename
+            fin_dynamics_time_constant
+            lift_constant
+            drag_constant
+            current_velocity_topic">
+    <joint name="${namespace}/fin${fin_id}_joint" type="revolute">
+        <limit effort="0" lower="${min_joint_limit}" upper="${max_joint_limit}" velocity="0"/>
+        <xacro:insert_block name="origin"/>
+        <!--<axis xyz="0 0 1"/>-->
         <axis xyz="0 1 0"/>
         <parent link="${parent_link}" />
@@ -132,52 +179,5 @@
         <origin xyz="0 0 0" rpy="0 0 0" />
         <geometry>
-          <mesh filename="${mesh_filename}" scale="1 1 1"/>
-        </geometry>
-      </visual>
-    </link>
-    <gazebo>
-      <plugin name="${namespace}_fin${fin_id}_model" filename="libuuv_fin_ros_plugin.so">
-        <dynamics>
-          <type>FirstOrder</type>
-          <timeConstant>${fin_dynamics_time_constant}</timeConstant>
-        </dynamics>
-        <liftdrag>
-          <type>Quadratic</type>
-          <lift_constant>${lift_constant}</lift_constant>
-          <drag_constant>${drag_constant}</drag_constant>
-        </liftdrag>
-        <current_velocity_topic>${current_velocity_topic}</current_velocity_topic>
-        <fin_id>${fin_id}</fin_id>
-        <link_name>${namespace}/fin${fin_id}</link_name>
-        <joint_name>${namespace}/fin${fin_id}_joint</joint_name>
-      </plugin>
-    </gazebo>
-  </xacro:macro>
-  <xacro:macro name="hor_right_fin_quadratic_macro"
-    params="namespace
-            parent_link
-            fin_id
-            *origin
-            min_joint_limit
-            max_joint_limit
-            mesh_filename
-            fin_dynamics_time_constant
-            lift_constant
-            drag_constant
-            current_velocity_topic">
-    <joint name="${namespace}/fin${fin_id}_joint" type="revolute">
-        <limit effort="0" lower="${min_joint_limit}" upper="${max_joint_limit}" velocity="0"/>
-        <xacro:insert_block name="origin"/>
-        <!--<axis xyz="0 0 1"/>-->
-        <axis xyz="0 -1 0"/>
-        <parent link="${parent_link}" />
-        <child link="${namespace}/fin${fin_id}" />
-    </joint>
-    <link name="${namespace}/fin${fin_id}">
-      <xacro:no_inertial />
-      <visual>
-        <origin xyz="0 0 0" rpy="0 0 0" />
-        <geometry>
-          <mesh filename="${mesh_filename}" scale="1 1 1"/>
+          <mesh filename="${mesh_filename}" scale="1 -1 1"/>
         </geometry>
       </visual>
@@ -216,4 +216,50 @@
         <limit effort="0" lower="${min_joint_limit}" upper="${max_joint_limit}" velocity="0"/>
         <xacro:insert_block name="origin"/>
+        <axis xyz="0 0 -1"/>
+        <parent link="${parent_link}" />
+        <child link="${namespace}/fin${fin_id}" />
+    </joint>
+    <link name="${namespace}/fin${fin_id}">
+      <xacro:no_inertial />
+      <visual>
+        <origin xyz="0 0 0" rpy="0 0 0" />
+        <geometry>
+          <mesh filename="${mesh_filename}" scale="1 1 1"/>
+        </geometry>
+      </visual>
+    </link>
+    <gazebo>
+      <plugin name="${namespace}_fin${fin_id}_model" filename="libuuv_fin_ros_plugin.so">
+        <dynamics>
+          <type>FirstOrder</type>
+          <timeConstant>${fin_dynamics_time_constant}</timeConstant>
+        </dynamics>
+        <liftdrag>
+          <type>Quadratic</type>
+          <lift_constant>${lift_constant}</lift_constant>
+          <drag_constant>${drag_constant}</drag_constant>
+        </liftdrag>
+        <current_velocity_topic>${current_velocity_topic}</current_velocity_topic>
+        <fin_id>${fin_id}</fin_id>
+        <link_name>${namespace}/fin${fin_id}</link_name>
+        <joint_name>${namespace}/fin${fin_id}_joint</joint_name>
+      </plugin>
+    </gazebo>
+  </xacro:macro>
+  <xacro:macro name="lat_down_fin_quadratic_macro"
+    params="namespace
+            parent_link
+            fin_id
+            *origin
+            min_joint_limit
+            max_joint_limit
+            mesh_filename
+            fin_dynamics_time_constant
+            lift_constant
+            drag_constant
+            current_velocity_topic">
+    <joint name="${namespace}/fin${fin_id}_joint" type="revolute">
+        <limit effort="0" lower="${min_joint_limit}" upper="${max_joint_limit}" velocity="0"/>
+        <xacro:insert_block name="origin"/>
         <axis xyz="0 0 1"/>
         <parent link="${parent_link}" />
@@ -247,49 +293,3 @@
     </gazebo>
   </xacro:macro>
-  <xacro:macro name="lat_down_fin_quadratic_macro"
-    params="namespace
-            parent_link
-            fin_id
-            *origin
-            min_joint_limit
-            max_joint_limit
-            mesh_filename
-            fin_dynamics_time_constant
-            lift_constant
-            drag_constant
-            current_velocity_topic">
-    <joint name="${namespace}/fin${fin_id}_joint" type="revolute">
-        <limit effort="0" lower="${min_joint_limit}" upper="${max_joint_limit}" velocity="0"/>
-        <xacro:insert_block name="origin"/>
-        <axis xyz="0 0 -1"/>
-        <parent link="${parent_link}" />
-        <child link="${namespace}/fin${fin_id}" />
-    </joint>
-    <link name="${namespace}/fin${fin_id}">
-      <xacro:no_inertial />
-      <visual>
-        <origin xyz="0 0 0" rpy="0 0 0" />
-        <geometry>
-          <mesh filename="${mesh_filename}" scale="1 1 1"/>
-        </geometry>
-      </visual>
-    </link>
-    <gazebo>
-      <plugin name="${namespace}_fin${fin_id}_model" filename="libuuv_fin_ros_plugin.so">
-        <dynamics>
-          <type>FirstOrder</type>
-          <timeConstant>${fin_dynamics_time_constant}</timeConstant>
-        </dynamics>
-        <liftdrag>
-          <type>Quadratic</type>
-          <lift_constant>${lift_constant}</lift_constant>
-          <drag_constant>${drag_constant}</drag_constant>
-        </liftdrag>
-        <current_velocity_topic>${current_velocity_topic}</current_velocity_topic>
-        <fin_id>${fin_id}</fin_id>
-        <link_name>${namespace}/fin${fin_id}</link_name>
-        <joint_name>${namespace}/fin${fin_id}_joint</joint_name>
-      </plugin>
-    </gazebo>
-  </xacro:macro>
 </robot>
